File: 32u4 sumo deneme kartı v1.1/32u4 denemesi.brd (EAGLE design)
At the start: 100 x 100 mm, 131 parts, among them IC1 IC_555-SOIC8, IC2 LM2577S, J1 AVR_SPI_PRG_6NS, Q6 SI3456BDVSOT-5-6, U1 TB6612FNG

Commit message: ver1.3
Parts:
- removed Q6: SI3456BDVSOT-5-6, m-pad-2.1:SOT23-6
- removed U$11: LM393, SparkFun-AnalogIC:SO08
- added IC3: LMV358MX, linear:SO08
- added Q2: SI3456BDVSOT-5-6, m-pad-2.1:SOT23-6
- added R45: 10k, SparkFun-Resistors:1206
- added R46, R50: 2.2k, SparkFun-Resistors:1206
- added S3: (no value), SparkFun-Electromechanical:SWITCH-SPDT
- added T2: (no value), zetex:SOT-23
- C1, C14, C15, C18, C19, C2, C20, C23, C24, C25, C26, C27, C28, C29, C3, C30, C34, C35, C36, C4, C5, C9: device SparkFun-Passives:0805 -> SparkFun-Passives:1206
- C13: device SparkFun-Capacitors:EIA3528 -> SparkFun-Passives:1206
- C16, C17, C8: device SparkFun-Capacitors:EIA3216 -> SparkFun-Passives:1206
- R1, R11, R13, R16, R17, R18, R19, R20, R21, R22, R23, R30, R33, R37, R40, R41, R42, R43, R44, R47, R6, R7, R8, R9: device SparkFun-Resistors:0805 -> SparkFun-Resistors:1206
- R10: value 10.4k -> 10.5k; device SparkFun-Resistors:0805 -> SparkFun-Resistors:1206
- R12: value 39.2k -> 39.2; device SparkFun-Passives:0402-RES -> SparkFun-Resistors:1206
- R14, R15: value 220 -> 1k; device SparkFun-Resistors:0805 -> SparkFun-Resistors:1206
- R2, R3: value 10K -> 10k; device SparkFun-Resistors:0805 -> SparkFun-Resistors:1206
- R26, R29, R32, R35: device SparkFun-Passives:0402-RES -> SparkFun-Resistors:1206
- R27: value 1k -> 4.7k; device SparkFun-Resistors:0805 -> SparkFun-Resistors:1206
- R36: value 10k -> 1k; device SparkFun-Resistors:0805 -> SparkFun-Resistors:1206
- R38: value 10k -> 7.5k; device SparkFun-Resistors:0805 -> SparkFun-Resistors:1206
- R39: value 10k -> 68k; device SparkFun-Resistors:0805 -> SparkFun-Resistors:1206
- R4, R5: value 4.7K -> 4.7k; device SparkFun-Resistors:0805 -> SparkFun-Resistors:1206
- R48: value 2.2k -> 100; device SparkFun-Resistors:0805 -> SparkFun-Resistors:1206
- R49: value 100 -> 4.7k; device SparkFun-Passives:0402-RES -> SparkFun-Resistors:1206
- S2: device switch:M9040P -> SparkFun-Electromechanical:SWITCH-SPDT
- moved R26 85.7 mm to (86.4, 90.6)
- moved R48 85.7 mm to (51.8, 94.6)
- moved R35 79.4 mm to (9.17, 67.7), turned to 0 degrees
- moved R29 77.7 mm to (94.8, 69.4), turned to 180 degrees
- moved C25 70.8 mm to (77.9, 91.0)
- moved R49 65.7 mm to (95.9, 56.5), turned to 180 degrees
- moved R32 57.5 mm to (19.8, 93.3), turned to 270 degrees
- moved C24 54.1 mm to (23.3, 89.5), turned to 0 degrees
- moved C21 46.8 mm to (29.2, 11.4), turned to 90 degrees
- moved C7 28.1 mm to (43.9, 53.0)
- moved C22 25.0 mm to (29.1, 17.4), turned to 270 degrees
- moved C5 24.7 mm to (35.5, 80.1), turned to 0 degrees
- moved R11 21.8 mm to (13.4, 20.8)
- moved C2 18.6 mm to (34.3, 61.7), turned to 270 degrees
- moved C23 17.9 mm to (8.38, 80.5)
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Connections:
- net N$13 renamed VSW
- removed net N$30: R22.2, U$6.VS
- removed net N$47: BATTERY.1, Q6.4
- removed net N$48: Q6.6, S2.2, S2.3
- new net N$49: BATTERY.1, Q2.1, Q2.2, Q2.5, Q2.6
- new net N$51: Q2.4, S2.3
- new net N$54: S2.1, S2.2, S3.2
- new net VS1: C23.1, R19.2, U$9.VS
- new net VS2: C24.1, R20.2, U$8.VS
- new net VS3: C25.1, R21.2, U$7.VS
- new net VS4: C26.1, R22.2, U$6.VS
- net +5V: now also C17.1, IC3.8, R14.1, R15.1, R16.1, R23.1, R40.2, R49.2, R9.1, T2.2; no longer C17.A, C23.1, C24.1, C25.1, C26.1, R14.2, R15.2, R16.2, R23.2, R27.2, R40.1, R9.2, U$11.8
- net 38KHZOUT: now also R48.2; no longer R49.1
- net D10: now also R36.2, R37.1; no longer R38.1, R39.2
- net D4: now also R9.2; no longer R9.1
- net D9: now also IC3.1; no longer U$11.1
- net GND: now also C13.2, C16.2, C17.2, C21.2, C22.2, C3.1, C4.1, C6.1, C7.1, C8.2, IC2.6, IC3.4, Q2.3, R18.2, R3.2, R37.2, R45.1, R50.1; no longer C13.C, C16.C, C17.C, C21.1, C22.1, C3.2, C4.2, C6.2, C7.2, C8.C, Q6.3, R18.1, R3.1, R39.1, U$11.4
- net N$1: now also C7.2; no longer C7.1
- net N$11: now also IC3.5, R27.1, R45.2; no longer R19.2, U$9.VS
- net N$15: now also R10.1; no longer R10.2
- net N$16: now also R48.1; no longer R49.2
- net N$17: now also R36.1, R38.1; no longer R37.1, R38.2
- net N$18: now also R38.2, R39.1; no longer R36.1, R37.2
- net N$19: now also C32.1, R40.1; no longer C32.2, R40.2
- net N$20: now also C32.2; no longer C32.1
- net N$21: now also IC3.2; no longer U$11.2
- net N$22: now also R14.2; no longer R14.1
- net N$23: now also R15.2; no longer R15.1
- net N$24: now also R16.2, R23.2; no longer R16.1, R23.1, R27.1
- net N$25: now also R18.1; no longer R18.2
- net N$26: now also IC3.6, R49.1, R50.2; no longer R20.2, U$8.VS
- net N$28: now also IC3.7, T2.3; no longer R21.2, U$7.VS
- net N$3: now also C6.2; no longer C6.1
- net N$34: now also R35.1; no longer R26.1
- net N$38: now also R32.1; no longer R29.1
- net N$4: now also C4.2, R1.2; no longer C4.1, R1.1
- net N$42: now also R26.1; no longer R32.1
- net N$46: now also R29.1; no longer R35.1
- net N$5: now also C3.2, R1.1; no longer C3.1, R1.2
- net N$50: now also IC3.3; no longer U$11.3
- net N$52: now also R46.1; no longer R48.2
- net N$53: now also R46.2; no longer R48.1
- net N$7: now also R3.1; no longer R3.2
- net N$8: now also R39.2; no longer R36.2
- net VIN: now also C21.1, S3.1; no longer C21.2, S2.1
- net VUSB: now also C8.1, T2.1; no longer C8.A
- net V_BATT: now also C13.1, C16.1, C22.1, R10.2, R27.2, S3.3; no longer C13.A, C16.A, C22.2, R10.1
Routing:
- net V_BATT: track 159.1 -> 252.8 mm, vias 6 -> 8
- net +5V: track 553.3 -> 618.1 mm, vias 9 -> 10
- net DRAIN: track 157.5 -> 106.6 mm, vias 0 -> 1
- net N$47: track 40.8 -> 0.00 mm
- net N$49: track 0.00 -> 40.7 mm
- net VIN: track 83.3 -> 43.1 mm
- net A5: track 84.3 -> 46.0 mm, vias 1 -> 3
- net N$28: track 4.45 -> 40.9 mm, vias 0 -> 2
- net MOSI: track 64.3 -> 100.3 mm, vias 1 -> 3
- net 2,6: track 11.3 -> 42.9 mm
- net MISO: track 53.3 -> 83.2 mm, vias 2 -> 4
- net D8: track 38.6 -> 67.2 mm, vias 5 -> 4
- net D7: track 24.4 -> 52.0 mm
- net D10: track 83.0 -> 109.9 mm, vias 4 -> 2
- net D-: track 87.5 -> 60.7 mm
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- added copper zone on layer 1, net GND
- added copper zone on layer 16, net GND
- added copper zone on layer 1, net N$30
