File: 32u4 sumo deneme kartı v1.1/32u4 denemesi.sch (EAGLE design)
At the start: 134 parts, among them IC1 IC_555-SOIC8, J1 AVR_SPI_PRG_6NS, Q1 BS170, Q2 BS170, Q3 BS170, Q4 BS170, Q5 FDD4141, U1 TB6612FNG

Commit message: ver1.1
Parts:
- removed C31: 100nF, SparkFun-Passives:CAP0805
- removed Q2, Q3, Q4: BS170, gm-trans:BS170
- removed Q5: FDD4141, transistor-fet:FDD4141TO252
- removed R45: 1k, SparkFun-Resistors:RESISTOR0805-RES
- removed R46: 3k, SparkFun-Resistors:RESISTOR0805-RES
- removed S3: (no value), SparkFun-Electromechanical:SWITCH-SPDTPTH
- added C37: 0.33uF, SparkFun-Passives:CAP1206
- added IC2: LM2577S, v-reg-3:LM2577S
- added Q6: SI3456BDVSOT-5-6, m-pad-2.1:SI3456BDVSOT-5-6
- added R48: 2.2k, SparkFun-Resistors:RESISTOR0805-RES
- added R49: 100, SparkFun-Passives:RESISTOR0402-RES
- C12: value 220uF -> 680uF
- D2: value S3A -> (none); device s3x_10:S3A -> m-pad-2.1:D_SCHOTTKYA
- Q1: value BS170 -> (none); device gm-trans:BS170 -> transistors:2N7000_SOT23
- R10: value 5k -> 10.4k
- R11: value 1k -> 2k
- R16: value 1.5k -> 1k
- R23, R27: value 10k -> 1k; device SparkFun-Passives:RESISTOR0402-RES -> SparkFun-Resistors:RESISTOR0805-RES
- R30: device SparkFun-Passives:RESISTOR0402-RES -> SparkFun-Resistors:RESISTOR0805-RES
- R33: value 10k -> 47k; device SparkFun-Passives:RESISTOR0402-RES -> SparkFun-Resistors:RESISTOR0805-RES
- U$4: value TO263-5L -> DMG1012UW; device m-pad-2.1:TO263-5L -> m-pad-2.1:DMG1012UW
- renumbered LED1 to PWRLED, LED2 to RXLED, LED3 to TXLED
Connections:
- removed net N$32: Q1.S, R25.S
- removed net N$36: Q2.S, R28.S
- removed net N$43: Q4.G, R33.2
- removed net N$44: Q4.S, R34.S
- removed net N$49: R45.1, R46.1, S1.S
- removed net N$51: Q3.D, S3.O, S3.P
- new net DRAIN: R25.S, R28.S, R31.S, R34.S, S4.S
- new net N$52: IC2.COMP, R48.2
- new net N$53: C37.1, R48.1
- net +5V: now also R23.2, R27.2, S1.P, S1.S; no longer C31.1, C8.+, C9.1
- net 38KHZOUT: now also R49.1; no longer R23.1, R27.1, R30.1, R33.1, S4.S
- net D11: now also U1.PWMA; no longer R17.1
- net D13: no longer LED4.C, R46.2
- net D5: now also R17.1; no longer U1.PWMA
- net GND: now also C37.2, IC2.GND, Q1.S, Q6.G, R33.1, U$4.S; no longer C31.2, Q1.D, Q2.D, Q4.D, Q5.G, S1.O, S1.P, S3.S, U$4.GND
- net N$13: now also IC2.VSW; no longer U$4.SW
- net N$15: now also IC2.FB; no longer U$4.FB
- net N$16: now also R49.2, U$4.G; no longer L2.1, S2.O, U$4.VIN
- net N$24: now also R23.1, R27.1; no longer R45.2
- net N$31: now also U$4.D; no longer Q1.G, R23.2
- net N$35: now also LED4.C, Q1.D; no longer Q2.G, R27.2
- net N$39: now also S1.O; no longer Q3.G
- net N$40: now also Q1.G, R30.1, R33.2; no longer Q3.S, R31.S
- net N$47: now also Q6.S; no longer Q5.D
- net N$48: now also Q6.D@3; no longer Q5.S
- net VIN: now also IC2.VIN, L2.1, S2.O
- net VUSB: now also C8.+, C9.1
Other:
- note added: "100uH"
- note added: "BOOST CONVERTER(LM2577)"
- note removed: "BOOST CONVERTER(XL6009)"

Commit message: ver1.3
Parts:
- removed Q6: SI3456BDVSOT-5-6, m-pad-2.1:SI3456BDVSOT-5-6
- removed U$11: LM393, SparkFun-AnalogIC:LM393
- added IC3: LMV358MX, linear:LMV358MX
- added Q2: SI3456BDVSOT-5-6, m-pad-2.1:SI3456BDVSOT-5-6
- added R45: 10k, SparkFun-Resistors:RESISTOR1206
- added R46, R50: 2.2k, SparkFun-Resistors:RESISTOR1206
- added S3: (no value), SparkFun-Electromechanical:SWITCH-SPDTPTH
- added T2: (no value), zetex:PMOSSOT23
- C1, C14, C15, C18, C19, C2, C20, C23, C24, C25, C26, C27, C28, C29, C3, C30, C34, C35, C36, C4, C5, C9: device SparkFun-Passives:CAP0805 -> SparkFun-Passives:CAP1206
- C13: device SparkFun-Capacitors:CAP_POL3528 -> SparkFun-Passives:CAP1206
- C16, C17, C8: device SparkFun-Capacitors:CAP_POL1206 -> SparkFun-Passives:CAP1206
- R1, R11, R13, R16, R17, R18, R19, R20, R21, R22, R23, R30, R33, R37, R40, R41, R42, R43, R44, R47, R6, R7, R8, R9: device SparkFun-Resistors:RESISTOR0805-RES -> SparkFun-Resistors:RESISTOR1206
- R10: value 10.4k -> 10.5k; device SparkFun-Resistors:RESISTOR0805-RES -> SparkFun-Resistors:RESISTOR1206
- R12: value 39.2k -> 39.2; device SparkFun-Passives:RESISTOR0402-RES -> SparkFun-Resistors:RESISTOR1206
- R14, R15: value 220 -> 1k; device SparkFun-Resistors:RESISTOR0805-RES -> SparkFun-Resistors:RESISTOR1206
- R2, R3: value 10K -> 10k; device SparkFun-Resistors:RESISTOR0805-RES -> SparkFun-Resistors:RESISTOR1206
- R26, R29, R32, R35: device SparkFun-Passives:RESISTOR0402-RES -> SparkFun-Resistors:RESISTOR1206
- R27: value 1k -> 4.7k; device SparkFun-Resistors:RESISTOR0805-RES -> SparkFun-Resistors:RESISTOR1206
- R36: value 10k -> 1k; device SparkFun-Resistors:RESISTOR0805-RES -> SparkFun-Resistors:RESISTOR1206
- R38: value 10k -> 7.5k; device SparkFun-Resistors:RESISTOR0805-RES -> SparkFun-Resistors:RESISTOR1206
- R39: value 10k -> 68k; device SparkFun-Resistors:RESISTOR0805-RES -> SparkFun-Resistors:RESISTOR1206
- R4, R5: value 4.7K -> 4.7k; device SparkFun-Resistors:RESISTOR0805-RES -> SparkFun-Resistors:RESISTOR1206
- R48: value 2.2k -> 100; device SparkFun-Resistors:RESISTOR0805-RES -> SparkFun-Resistors:RESISTOR1206
- R49: value 100 -> 4.7k; device SparkFun-Passives:RESISTOR0402-RES -> SparkFun-Resistors:RESISTOR1206
- S2: device switch:M9040P -> SparkFun-Electromechanical:SWITCH-SPDTPTH
Connections:
- net N$13 renamed VSW
- removed net N$30: R22.2, U$6.VS
- removed net N$47: BATTERY-1.KL, Q6.S
- removed net N$48: Q6.D@3, S2.P, S2.S
- new net N$49: BATTERY-1.KL, Q2.D
- new net N$51: Q2.S, S2.S
- new net N$54: S2.O, S2.P, S3.P
- new net VS1: C23.1, R19.2, U$9.VS
- new net VS2: C24.1, R20.2, U$8.VS
- new net VS3: C25.1, R21.2, U$7.VS
- new net VS4: C26.1, R22.2, U$6.VS
- net +5V: now also C17.1, IC3P.V+, R14.1, R15.1, R16.1, R23.1, R40.2, R49.2, R9.1, T2.S; no longer C17.+, C23.1, C24.1, C25.1, C26.1, R14.2, R15.2, R16.2, R23.2, R27.2, R40.1, R9.2, U$11G1.V+
- net 38KHZOUT: now also R48.2; no longer R49.1
- net D10: now also R36.2, R37.1; no longer R38.1, R39.2
- net D4: now also R9.2; no longer R9.1
- net D9: now also IC3A.OUT; no longer U$11G1.OUT
- net GND: now also C13.2, C16.2, C17.2, C21.2, C22.2, C3.1, C4.1, C6.1, C7.1, C8.2, IC3P.V-, Q2.G, R18.2, R3.2, R37.2, R45.1, R50.1; no longer C13.-, C16.-, C17.-, C21.1, C22.1, C3.2, C4.2, C6.2, C7.2, C8.-, Q6.G, R18.1, R3.1, R39.1, U$11G1.V-
- net N$1: now also C7.2; no longer C7.1
- net N$11: now also IC3B.+IN, R27.1, R45.2; no longer R19.2, U$9.VS
- net N$15: now also R10.1; no longer R10.2
- net N$16: now also R48.1; no longer R49.2
- net N$17: now also R36.1, R38.1; no longer R37.1, R38.2
- net N$18: now also R38.2, R39.1; no longer R36.1, R37.2
- net N$19: now also C32.1, R40.1; no longer C32.2, R40.2
- net N$20: now also C32.2; no longer C32.1
- net N$21: now also IC3A.-IN; no longer U$11G1.-IN
- net N$22: now also R14.2; no longer R14.1
- net N$23: now also R15.2; no longer R15.1
- net N$24: now also R16.2, R23.2; no longer R16.1, R23.1, R27.1
- net N$25: now also R18.1; no longer R18.2
- net N$26: now also IC3B.-IN, R49.1, R50.2; no longer R20.2, U$8.VS
- net N$28: now also IC3B.OUT, T2.G; no longer R21.2, U$7.VS
- net N$3: now also C6.2; no longer C6.1
- net N$34: now also R35.1; no longer R26.1
- net N$38: now also R32.1; no longer R29.1
- net N$4: now also C4.2, R1.2; no longer C4.1, R1.1
- net N$42: now also R26.1; no longer R32.1
- net N$46: now also R29.1; no longer R35.1
- net N$5: now also C3.2, R1.1; no longer C3.1, R1.2
- net N$50: now also IC3A.+IN; no longer U$11G1.+IN
- net N$52: now also R46.1; no longer R48.2
- net N$53: now also R46.2; no longer R48.1
- net N$7: now also R3.1; no longer R3.2
- net N$8: now also R39.2; no longer R36.2
- net VIN: now also C21.1, S3.O; no longer C21.2, S2.O
- net VUSB: now also C8.1, T2.D; no longer C8.+
- net V_BATT: now also C13.1, C16.1, C22.1, R10.2, R27.2, S3.S; no longer C13.+, C16.+, C22.2, R10.1
Other:
- note added: "+5v AUTO SELECTOR"
